Commit message: Gen3 6-DOF: joint 2/3/5 limits from the arm's own fault thresholds
The URDF had 2.24 / 2.57 / 2.09 rad, about the actuators' warning
thresholds. The arm faults only at 138.08 / 152.41 / 127.77 deg (each
actuator's JOINT_LIMIT_HIGH/LOW error threshold, read over Kortex
2026-10-15). With its own margin and slow zone on top, the hand-guidance
controller froze the whole arm 5-7 deg short of what the arm allows, e.g.
joint 3 at -145.5 deg, close to Kinova's own poses. The limits are now the
fault thresholds minus 2 deg: 2.3751 / 2.6251 / 2.1951 rad.

Co-Authored-By: Claude Opus 5.5 (1M context) <noreply@anthropic.com>
Claude-Session: https://claude.ai/code/session_01Jfx6mvvRwpNWQoXTYJGZJY

File: kortex_description/arms/gen3/6dof/urdf/gen3_macro.xacro (robot description, xacro)
@@ -174,5 +174,6 @@
       <child link="${prefix}bicep_link" />
       <axis xyz="0 0 1" />
-      <limit lower="-2.24" upper="2.24" effort="39" velocity="1.3963" />
+      <!-- joint_2: the arm's own fault threshold is 138.08 deg (actuator safety JOINT_LIMIT_HIGH/LOW error threshold, read 2026-10-15; its warning is lower). Was 2.24 rad, about the warning: our controller then froze the arm 5-7 deg short of what the arm allows. Fault minus 2 deg. -->
+      <limit lower="-2.3751" upper="2.3751" effort="39" velocity="1.3963" />
     </joint>
     <link name="${prefix}forearm_link">
@@ -203,5 +204,6 @@
       <child link="${prefix}forearm_link" />
       <axis xyz="0 0 1" />
-      <limit lower="-2.57" upper="2.57" effort="39" velocity="1.3963" />
+      <!-- joint_3: the arm's own fault threshold is 152.41 deg (actuator safety JOINT_LIMIT_HIGH/LOW error threshold, read 2026-10-15; its warning is lower). Was 2.57 rad, about the warning: our controller then froze the arm 5-7 deg short of what the arm allows. Fault minus 2 deg. -->
+      <limit lower="-2.6251" upper="2.6251" effort="39" velocity="1.3963" />
     </joint>
     <link name="${prefix}spherical_wrist_1_link">
@@ -272,5 +274,6 @@
       <child link="${prefix}spherical_wrist_2_link" />
       <axis xyz="0 0 1" />
-      <limit lower="-2.09" upper="2.09" effort="9" velocity="1.2218" />
+      <!-- joint_5: the arm's own fault threshold is 127.77 deg (actuator safety JOINT_LIMIT_HIGH/LOW error threshold, read 2026-10-15; its warning is lower). Was 2.09 rad, about the warning: our controller then froze the arm 5-7 deg short of what the arm allows. Fault minus 2 deg. -->
+      <limit lower="-2.1951" upper="2.1951" effort="9" velocity="1.2218" />
     </joint>
     <xacro:if value="${vision}">

Commit message: Gen3 6-DOF: joint 2/3/5 limits from the arm's own fault thresholds
The URDF's limits sat about at the arm's warnings, 5-7 deg short of where it
faults: the controller froze the arm there. Each is now the arm's fault
threshold minus 2 deg (actuator safety JOINT_LIMIT_HIGH/LOW, read
2026-10-15): joint_2 138.08 deg, joint_3 152.41, joint_5 127.77.
On jazzy-rackthor's file (CRLF, with the torque work); e38d97b's change.

Co-Authored-By: Claude Opus 5.5 (1M context) <noreply@anthropic.com>
Claude-Session: https://claude.ai/code/session_01Jfx6mvvRwpNWQoXTYJGZJY

File: kortex_description/arms/gen3/6dof/urdf/gen3_macro.xacro (robot description, xacro)
@@ -174,5 +174,6 @@
       <child link="${prefix}bicep_link" />
       <axis xyz="0 0 1" />
-      <limit lower="-2.24" upper="2.24" effort="39" velocity="1.3963" />
+      <!-- joint_2: the arm's own fault threshold is 138.08 deg (actuator safety JOINT_LIMIT_HIGH/LOW error threshold, read 2026-10-15; its warning is lower). Was 2.24 rad, about the warning: our controller then froze the arm 5-7 deg short of what the arm allows. Fault minus 2 deg. -->
+      <limit lower="-2.3751" upper="2.3751" effort="39" velocity="1.3963" />
     </joint>
     <link name="${prefix}forearm_link">
@@ -199,5 +200,6 @@
       <child link="${prefix}forearm_link" />
       <axis xyz="0 0 1" />
-      <limit lower="-2.57" upper="2.57" effort="39" velocity="1.3963" />
+      <!-- joint_3: the arm's own fault threshold is 152.41 deg (actuator safety JOINT_LIMIT_HIGH/LOW error threshold, read 2026-10-15; its warning is lower). Was 2.57 rad, about the warning: our controller then froze the arm 5-7 deg short of what the arm allows. Fault minus 2 deg. -->
+      <limit lower="-2.6251" upper="2.6251" effort="39" velocity="1.3963" />
     </joint>
     <link name="${prefix}spherical_wrist_1_link">
@@ -260,5 +262,6 @@
       <child link="${prefix}spherical_wrist_2_link" />
       <axis xyz="0 0 1" />
-      <limit lower="-2.09" upper="2.09" effort="9" velocity="1.2218" />
+      <!-- joint_5: the arm's own fault threshold is 127.77 deg (actuator safety JOINT_LIMIT_HIGH/LOW error threshold, read 2026-10-15; its warning is lower). Was 2.09 rad, about the warning: our controller then froze the arm 5-7 deg short of what the arm allows. Fault minus 2 deg. -->
+      <limit lower="-2.1951" upper="2.1951" effort="9" velocity="1.2218" />
     </joint>
     <xacro:if value="${vision}">

Commit message: kortex_driver: per-joint kinematic calibration (joint_offset, joint_compliance)
Optional <param>s of each arm <joint> in the ros2_control block:
joint_offset (rad) and joint_compliance (rad/(N*m)), both default 0.
rackthor's omnicalibrator fits them from hand-eye board views.

  reading:           q = q_raw + offset + compliance * tau
  position command:  q_raw_cmd = q_cmd - offset - compliance * tau_now

tau is the effort state as the interface reports it (N*m, ROS sign); for
commands, the last read. Velocity and effort commands and states are
unchanged, and the endless joints wrap as before ([-pi, pi] in, [0, 360)
deg out). Hold positions (activation, mode switches, leaving torque mode)
go through the same transform, so nothing jumps. The applied values are
logged once at init. Nothing is ever written to the actuators' own zero:
only readings and commands are translated.

Inert without the params: the default robot, mock, Gazebo and Isaac get
none (kortex_description emits them for the real driver only, from the
new joint_offsets / joint_compliance dicts, {joint_N: value}, passed
through load_robot -> load_arm -> kortex_ros2_control; gen3_lite accepts
and ignores them).

Not covered, by design:
- Twist mode (Kinova's internal Cartesian control) runs the arm's own
  kinematics on raw joints and cannot be corrected.
- Joint limits stay raw: the arm faults on its own thresholds while the
  URDF limits are compared with calibrated angles, so each limit moves
  by -offset. The offsets are under 2 deg and the URDF limits keep 2+ deg
  of margin inside the arm's thresholds.

The transform is a header-only pure function (joint_calibration.hpp)
with a gtest, including parsing the params from a ros2_control block.

Co-Authored-By: Claude Opus 5.5 (1M context) <noreply@anthropic.com>
Claude-Session: https://claude.ai/code/session_01Jfx6mvvRwpNWQoXTYJGZJY

File: kortex_description/arms/gen3/6dof/urdf/gen3_macro.xacro (robot description, xacro)
@@ -40,4 +40,6 @@
     gripper_max_force:=100.0
     effort_command_signs:=''
+    joint_offsets:=${dict()}
+    joint_compliance:=${dict()}
     use_fake_hardware:=false
     fake_sensor_commands:=false
@@ -72,4 +74,6 @@
       gripper_max_force="${gripper_max_force}"
       effort_command_signs="${effort_command_signs}"
+      joint_offsets="${joint_offsets}"
+      joint_compliance="${joint_compliance}"
       gripper_joint_name="${gripper_joint_name}"
       gripper="${gripper}"/>

File: kortex_description/arms/gen3/6dof/urdf/kortex.ros2_control.xacro (robot description, xacro)
@@ -1,4 +1,16 @@
 <?xml version="1.0"?>
 <robot xmlns:xacro="http://www.ros.org/wiki/xacro">
+  <!-- Per-joint kinematic calibration for kortex_driver (see its joint_calibration.hpp):
+       joint_offsets {joint_N: rad} and joint_compliance {joint_N: rad/(N*m)}, unprefixed joint
+       names, become the joint's joint_offset / joint_compliance params. The real driver only:
+       nothing is emitted for mock, Gazebo or Isaac. A joint without an entry stays raw. -->
+  <xacro:macro name="kortex_joint_calibration" params="joint joint_offsets joint_compliance">
+    <xacro:if value="${joint in joint_offsets}">
+      <param name="joint_offset">${joint_offsets[joint]}</param>
+    </xacro:if>
+    <xacro:if value="${joint in joint_compliance}">
+      <param name="joint_compliance">${joint_compliance[joint]}</param>
+    </xacro:if>
+  </xacro:macro>
   <xacro:macro name="kortex_ros2_control" params="
     name
@@ -25,4 +37,6 @@
     gripper_max_force:=100.0
     effort_command_signs:=''
+    joint_offsets:=${dict()}
+    joint_compliance:=${dict()}
     moveit_active:=false">
     <ros2_control name="${name}" type="system">
@@ -73,4 +87,8 @@
         <state_interface name="velocity"/>
         <state_interface name="effort"/>
+        <xacro:unless value="${use_fake_hardware or sim_gazebo or sim_isaac}">
+          <xacro:kortex_joint_calibration joint="joint_1"
+            joint_offsets="${joint_offsets}" joint_compliance="${joint_compliance}"/>
+        </xacro:unless>
       </joint>
       <joint name="${prefix}joint_2">
@@ -89,4 +107,8 @@
         <state_interface name="velocity"/>
         <state_interface name="effort"/>
+        <xacro:unless value="${use_fake_hardware or sim_gazebo or sim_isaac}">
+          <xacro:kortex_joint_calibration joint="joint_2"
+            joint_offsets="${joint_offsets}" joint_compliance="${joint_compliance}"/>
+        </xacro:unless>
       </joint>
       <joint name="${prefix}joint_3">
@@ -105,4 +127,8 @@
         <state_interface name="velocity"/>
         <state_interface name="effort"/>
+        <xacro:unless value="${use_fake_hardware or sim_gazebo or sim_isaac}">
+          <xacro:kortex_joint_calibration joint="joint_3"
+            joint_offsets="${joint_offsets}" joint_compliance="${joint_compliance}"/>
+        </xacro:unless>
       </joint>
       <joint name="${prefix}joint_4">
@@ -121,4 +147,8 @@
         <state_interface name="velocity"/>
         <state_interface name="effort"/>
+        <xacro:unless value="${use_fake_hardware or sim_gazebo or sim_isaac}">
+          <xacro:kortex_joint_calibration joint="joint_4"
+            joint_offsets="${joint_offsets}" joint_compliance="${joint_compliance}"/>
+        </xacro:unless>
       </joint>
       <joint name="${prefix}joint_5">
@@ -137,4 +167,8 @@
         <state_interface name="velocity"/>
         <state_interface name="effort"/>
+        <xacro:unless value="${use_fake_hardware or sim_gazebo or sim_isaac}">
+          <xacro:kortex_joint_calibration joint="joint_5"
+            joint_offsets="${joint_offsets}" joint_compliance="${joint_compliance}"/>
+        </xacro:unless>
       </joint>
       <joint name="${prefix}joint_6">
@@ -153,4 +187,8 @@
         <state_interface name="velocity"/>
         <state_interface name="effort"/>
+        <xacro:unless value="${use_fake_hardware or sim_gazebo or sim_isaac}">
+          <xacro:kortex_joint_calibration joint="joint_6"
+            joint_offsets="${joint_offsets}" joint_compliance="${joint_compliance}"/>
+        </xacro:unless>
       </joint>
       <xacro:unless value="${use_fake_hardware or sim_gazebo or sim_isaac}">

File: kortex_description/arms/gen3/7dof/urdf/gen3_macro.xacro (robot description, xacro)
@@ -22,4 +22,6 @@
     gripper_max_force:=100.0
     effort_command_signs:=''
+    joint_offsets:=${dict()}
+    joint_compliance:=${dict()}
     use_fake_hardware:=false
     fake_sensor_commands:=false
@@ -54,4 +56,6 @@
       gripper_max_force="${gripper_max_force}"
       effort_command_signs="${effort_command_signs}"
+      joint_offsets="${joint_offsets}"
+      joint_compliance="${joint_compliance}"
       gripper_joint_name="${gripper_joint_name}"
       gripper="${gripper}"/>

File: kortex_description/arms/gen3/7dof/urdf/kortex.ros2_control.xacro (robot description, xacro)
@@ -1,4 +1,16 @@
 <?xml version="1.0"?>
 <robot xmlns:xacro="http://www.ros.org/wiki/xacro">
+  <!-- Per-joint kinematic calibration for kortex_driver (see its joint_calibration.hpp):
+       joint_offsets {joint_N: rad} and joint_compliance {joint_N: rad/(N*m)}, unprefixed joint
+       names, become the joint's joint_offset / joint_compliance params. The real driver only:
+       nothing is emitted for mock, Gazebo or Isaac. A joint without an entry stays raw. -->
+  <xacro:macro name="kortex_joint_calibration" params="joint joint_offsets joint_compliance">
+    <xacro:if value="${joint in joint_offsets}">
+      <param name="joint_offset">${joint_offsets[joint]}</param>
+    </xacro:if>
+    <xacro:if value="${joint in joint_compliance}">
+      <param name="joint_compliance">${joint_compliance[joint]}</param>
+    </xacro:if>
+  </xacro:macro>
   <xacro:macro name="kortex_ros2_control" params="
     name
@@ -25,4 +37,6 @@
     gripper_max_force:=100.0
     effort_command_signs:=''
+    joint_offsets:=${dict()}
+    joint_compliance:=${dict()}
     moveit_active:=false">
     <ros2_control name="${name}" type="system">
@@ -73,4 +87,8 @@
         <state_interface name="velocity"/>
         <state_interface name="effort"/>
+        <xacro:unless value="${use_fake_hardware or sim_gazebo or sim_isaac}">
+          <xacro:kortex_joint_calibration joint="joint_1"
+            joint_offsets="${joint_offsets}" joint_compliance="${joint_compliance}"/>
+        </xacro:unless>
       </joint>
       <joint name="${prefix}joint_2">
@@ -89,4 +107,8 @@
         <state_interface name="velocity"/>
         <state_interface name="effort"/>
+        <xacro:unless value="${use_fake_hardware or sim_gazebo or sim_isaac}">
+          <xacro:kortex_joint_calibration joint="joint_2"
+            joint_offsets="${joint_offsets}" joint_compliance="${joint_compliance}"/>
+        </xacro:unless>
       </joint>
       <joint name="${prefix}joint_3">
@@ -105,4 +127,8 @@
         <state_interface name="velocity"/>
         <state_interface name="effort"/>
+        <xacro:unless value="${use_fake_hardware or sim_gazebo or sim_isaac}">
+          <xacro:kortex_joint_calibration joint="joint_3"
+            joint_offsets="${joint_offsets}" joint_compliance="${joint_compliance}"/>
+        </xacro:unless>
       </joint>
       <joint name="${prefix}joint_4">
@@ -121,4 +147,8 @@
         <state_interface name="velocity"/>
         <state_interface name="effort"/>
+        <xacro:unless value="${use_fake_hardware or sim_gazebo or sim_isaac}">
+          <xacro:kortex_joint_calibration joint="joint_4"
+            joint_offsets="${joint_offsets}" joint_compliance="${joint_compliance}"/>
+        </xacro:unless>
       </joint>
       <joint name="${prefix}joint_5">
@@ -137,4 +167,8 @@
         <state_interface name="velocity"/>
         <state_interface name="effort"/>
+        <xacro:unless value="${use_fake_hardware or sim_gazebo or sim_isaac}">
+          <xacro:kortex_joint_calibration joint="joint_5"
+            joint_offsets="${joint_offsets}" joint_compliance="${joint_compliance}"/>
+        </xacro:unless>
       </joint>
       <joint name="${prefix}joint_6">
@@ -153,4 +187,8 @@
         <state_interface name="velocity"/>
         <state_interface name="effort"/>
+        <xacro:unless value="${use_fake_hardware or sim_gazebo or sim_isaac}">
+          <xacro:kortex_joint_calibration joint="joint_6"
+            joint_offsets="${joint_offsets}" joint_compliance="${joint_compliance}"/>
+        </xacro:unless>
       </joint>
       <joint name="${prefix}joint_7">
@@ -169,4 +207,8 @@
         <state_interface name="velocity"/>
         <state_interface name="effort"/>
+        <xacro:unless value="${use_fake_hardware or sim_gazebo or sim_isaac}">
+          <xacro:kortex_joint_calibration joint="joint_7"
+            joint_offsets="${joint_offsets}" joint_compliance="${joint_compliance}"/>
+        </xacro:unless>
       </joint>
       <xacro:unless value="${use_fake_hardware or sim_gazebo or sim_isaac}">

File: kortex_description/arms/gen3_lite/6dof/urdf/gen3_lite_macro.xacro (robot description, xacro)
@@ -22,4 +22,6 @@
     gripper_max_force:=100.0
     effort_command_signs:=''
+    joint_offsets:=${dict()}
+    joint_compliance:=${dict()}
     use_fake_hardware:=false
     fake_sensor_commands:=false

File: kortex_description/robots/kortex_robot.xacro (robot description, xacro)
@@ -29,4 +29,6 @@
     gripper_max_force:=100.0
     effort_command_signs:=''
+    joint_offsets:=${dict()}
+    joint_compliance:=${dict()}
     gripper_com_port:=/dev/ttyUSB0
     moveit_active:=false">
@@ -58,4 +60,6 @@
       gripper_max_force="${gripper_max_force}"
       effort_command_signs="${effort_command_signs}"
+      joint_offsets="${joint_offsets}"
+      joint_compliance="${joint_compliance}"
       use_external_cable="${use_external_cable}"
       initial_positions="${initial_positions}"

Commit message: kortex_description gen3 6-DOF: joint origins from outside (kortex_joint_origins)
The arm's kinematic calibration, link geometry: define kortex_joint_origins
before load_robot as {joint: {xyz: [m], rpy: [rad]}} and those joints'
origins replace the nominal ones; joints left out, or the property left
undefined, keep upstream's. The same pattern as kortex_inertials.

rackthor passes arm.joint_origins from the robot's payload_calibration.yaml
(the omnicalibrator's L3 fit), real arm only. With nothing defined the
expanded URDF is byte-identical to before.

Co-Authored-By: Claude Opus 5.5 (1M context) <noreply@anthropic.com>
Claude-Session: https://claude.ai/code/session_01Ehy81z81Nvu46CnnmMbBXz

File: kortex_description/arms/gen3/6dof/urdf/gen3_macro.xacro (robot description, xacro)
@@ -11,4 +11,16 @@
        CAD values below stand, as upstream. -->
   <xacro:property name="kortex_inertials" default=""/>
+  <!-- Per-joint origins from outside (the arm's kinematic calibration):
+       define kortex_joint_origins before load_robot as {joint: {xyz: [x, y, z]
+       (m), rpy: [r, p, y] (rad)}}, unprefixed joint names, each the joint's
+       whole origin (parent link -> joint frame), replacing the nominal one
+       below. Joints left out keep theirs. Left undefined, all nominal, as
+       upstream. (rackthor: arm.joint_origins in the robot's
+       payload_calibration.yaml, from the omnicalibrator's link-geometry fit.) -->
+  <xacro:property name="kortex_joint_origins" default=""/>
+  <xacro:macro name="kortex_origin" params="joint xyz rpy">
+    <xacro:property name="o" value="${dict() if kortex_joint_origins == '' else (kortex_joint_origins.get(joint) or dict())}"/>
+    <origin xyz="${' '.join(map(str, o['xyz'])) if 'xyz' in o else xyz}" rpy="${' '.join(map(str, o['rpy'])) if 'rpy' in o else rpy}" />
+  </xacro:macro>
   <xacro:macro name="kortex_inertial" params="link xyz mass ixx ixy ixz iyy iyz izz">
     <xacro:property name="cad" value="${kortex_inertials == ''}"/>
@@ -174,5 +186,5 @@
     </link>
     <joint name="${prefix}joint_2" type="revolute">
-      <origin xyz="0 0.005375 -0.12838" rpy="1.5708 0.0 0.0" />
+      <xacro:kortex_origin joint="joint_2" xyz="0 0.005375 -0.12838" rpy="1.5708 0.0 0.0"/>
       <parent link="${prefix}shoulder_link" />
       <child link="${prefix}bicep_link" />
@@ -200,5 +212,5 @@
     </link>
     <joint name="${prefix}joint_3" type="revolute">
-      <origin xyz="0 -0.41 0" rpy="3.1416 0 0" />
+      <xacro:kortex_origin joint="joint_3" xyz="0 -0.41 0" rpy="3.1416 0 0"/>
       <parent link="${prefix}bicep_link" />
       <child link="${prefix}forearm_link" />
@@ -227,5 +239,5 @@
     <xacro:if value="${use_external_cable}">
       <joint name="${prefix}joint_4" type="revolute">
-        <origin xyz="0 0.20843 -0.006375" rpy="1.5708 0.0 0.0" />
+        <xacro:kortex_origin joint="joint_4" xyz="0 0.20843 -0.006375" rpy="1.5708 0.0 0.0"/>
         <parent link="${prefix}forearm_link" />
         <child link="${prefix}spherical_wrist_1_link" />
@@ -236,5 +248,5 @@
     <xacro:unless value="${use_external_cable}">
       <joint name="${prefix}joint_4" type="continuous">
-        <origin xyz="0 0.20843 -0.006375" rpy="1.5708 0.0 0.0" />
+        <xacro:kortex_origin joint="joint_4" xyz="0 0.20843 -0.006375" rpy="1.5708 0.0 0.0"/>
         <parent link="${prefix}forearm_link" />
         <child link="${prefix}spherical_wrist_1_link" />
@@ -262,5 +274,5 @@
     </link>
     <joint name="${prefix}joint_5" type="revolute">
-      <origin xyz="0 -0.00017505 -0.10593" rpy="-1.5708 0.0 0.0" />
+      <xacro:kortex_origin joint="joint_5" xyz="0 -0.00017505 -0.10593" rpy="-1.5708 0.0 0.0"/>
       <parent link="${prefix}spherical_wrist_1_link" />
       <child link="${prefix}spherical_wrist_2_link" />
@@ -311,5 +323,5 @@
     <xacro:if value="${use_external_cable}">
       <joint name="${prefix}joint_6" type="revolute">
-        <origin xyz="0 0.10593 -0.00017505" rpy="1.5708 0.0 0.0" />
+        <xacro:kortex_origin joint="joint_6" xyz="0 0.10593 -0.00017505" rpy="1.5708 0.0 0.0"/>
         <parent link="${prefix}spherical_wrist_2_link" />
         <child link="${prefix}bracelet_link" />
@@ -320,5 +332,5 @@
     <xacro:unless value="${use_external_cable}">
       <joint name="${prefix}joint_6" type="continuous">
-        <origin xyz="0 0.10593 -0.00017505" rpy="1.5708 0.0 0.0" />
+        <xacro:kortex_origin joint="joint_6" xyz="0 0.10593 -0.00017505" rpy="1.5708 0.0 0.0"/>
         <parent link="${prefix}spherical_wrist_2_link" />
         <child link="${prefix}bracelet_link" />
